File: hardware/esp32-ethernet-warp.kicad_pcb (KiCad board)
At the start: 4 copper layers, 104 x 42 mm, 117 parts, among them J201 TJLC_001LA1, P101 FLASH, P201 CON-SENSOR2, P202 CON-SENSOR2, P205 CON-SENSOR2, P206 CON-SENSOR2, Q101 BC817, Q102 BC817, SW101 B3U-1000P, SW102 B3U-1000P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

Commit message: mark C314 as DNP
Parts:
- C314: value 1nF/2kV -> DNP
Changed lines of the file:
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@@
         (effects (font (size 0.3 0.3) (thickness 0.075)))
     )
-    (fp_text value "1nF/2kV" (at 0 -0.65) (layer "F.Fab")
+    (fp_text value "DNP" (at 0 -0.65) (layer "F.Fab")
         (effects (font (size 0.3 0.3) (thickness 0.075)))
     )
