File: hardware/ethernet.kicad_sch (KiCad schematic)
At the start: 36 parts, among them J201 TJLC_001LA1, U301 KSZ8091RNACA, U404 TPD4S010DQA, X301 25Mhz-10pF

Commit message: mark C314 as DNP
Parts:
- C314: value 1nF/2kV -> DNP
Changed lines of the file:
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@@
   (title_block
     (title "WARP ESP32 Ethernet Brick")
-    (date "2023-12-27")
+    (date "2024-02-01")
     (rev "1.3")
     (company "Tinkerforge GmbH")
@@
       (effects (font (size 1.27 1.27)) (justify left))
     )
-    (property "Value" "1nF/2kV" (at 252.73 78.74 90)
+    (property "Value" "DNP" (at 252.73 78.74 90)
       (effects (font (size 1.27 1.27)) (justify left))
     )
